File: filpilote/esp_pilote.sch (EAGLE design)
At the start: 22 parts, among them IC1 ACS758LCB-050B-PFF-T

Commit message: Mise à jour PCB
Parts:
- removed JP2, JP4, JP5: (no value), pinhead:PINHD-1X1
- added R5, R6, R7, R8: 10k, rcl:R-EU_0204/7
- JP1, JP3: device pinhead:PINHD-1X1 -> pinhead:PINHD-1X2
- U$4: value HLK-PM03 -> MAINS_CONVERTERS
Connections:
- removed net VCC+3.3V: C1.1, IC1.VCC, MDL1.VCC, R3.1, SV1.1, U$3.VCC, U$4.VO+
- new net N$16: MDL1.CH_PD, R8.2
- new net N$18: MDL1.GPIO15, R7.1
- new net VCC: C1.1, IC1.VCC, MDL1.VCC, R3.1, R6.2, SV1.1, U$4.VO+
- net GND: now also JP3.2, R5.1, R7.2, R8.1
- net N$13: now also MDL1.RESET, R5.2; no longer JP4.1, MDL1.CH_PD
- net N$15: now also JP1.2; no longer JP2.1
- net N$17: now also MDL1.GPIO2, R6.1; no longer JP5.1, MDL1.RESET
- net N$9: now also MDL1.GPIO16; no longer MDL1.GPIO15

Commit message: Correction pcb
Connections:
- net N$9 renamed DS18B20
- net GND: no longer R8.1
- net VCC: now also R8.1, U$3.VCC
Changed lines of the file:
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@@
 <pinref part="SV1" gate="G$1" pin="1"/>
 <wire x1="-10.16" y1="50.8" x2="-25.4" y2="50.8" width="0.1524" layer="91"/>
+<pinref part="R8" gate="G$1" pin="1"/>
+<wire x1="0" y1="55.88" x2="0" y2="43.18" width="0.1524" layer="91"/>
 </segment>
 <segment>
@@
 <wire x1="-7.62" y1="109.22" x2="0" y2="109.22" width="0.1524" layer="91"/>
 <junction x="0" y="109.22"/>
+<pinref part="U$3" gate="G$1" pin="VCC"/>
+<wire x1="7.62" y1="93.98" x2="0" y2="93.98" width="0.1524" layer="91"/>
+<wire x1="0" y1="93.98" x2="0" y2="109.22" width="0.1524" layer="91"/>
 </segment>
 </net>
@@
 <wire x1="-5.08" y1="60.96" x2="-5.08" y2="88.9" width="0.1524" layer="91"/>
 <junction x="-5.08" y="88.9"/>
-<pinref part="R8" gate="G$1" pin="1"/>
-<wire x1="0" y1="55.88" x2="0" y2="60.96" width="0.1524" layer="91"/>
-<junction x="0" y="60.96"/>
 </segment>
 </net>
@@
 </segment>
 </net>
-<net name="N$9" class="0">
+<net name="DS18B20" class="0">
 <segment>
 <pinref part="R3" gate="G$1" pin="2"/>
