File: filpilote/esp_pilote.brd (EAGLE design)
At the start: 56 x 79 mm, 22 parts, among them IC1 ACS758LCB-050B-PFF-T

Commit message: Mise à jour PCB
Parts:
- removed JP2, JP4, JP5: (no value), pinhead:1X01
- added R5, R6, R7, R8: 10k, rcl:0204/7
- JP1, JP3: device pinhead:1X01 -> pinhead:1X02
- U$4: value HLK-PM03 -> MAINS_CONVERTERS
- moved R3 25.9 mm to (6.79, 66.5), turned to 90 degrees
- moved U$3 2.97 mm to (35.3, 59.2), turned to 180 degrees
- moved C1 2.43 mm to (34.3, 51.8), turned to 270 degrees
- moved JP3 2.24 mm to (33.0, 69.0)
- moved MDL1 2.00 mm to (17.5, 70.4)
- moved JP1 1.58 mm to (32.0, 76.0), turned to 270 degrees
- moved SV1 1.12 mm to (4.09, 65.4)
Connections:
- removed net VCC+3.3V: C1.1, IC1.1, MDL1.VCC, R3.1, SV1.1, U$3.3, U$4.VO+
- new net N$16: MDL1.CH_PD, R8.2
- new net N$18: MDL1.GPIO15, R7.1
- new net VCC: C1.1, IC1.1, MDL1.VCC, R3.1, R6.2, SV1.1, U$4.VO+
- net GND: now also JP3.2, R5.1, R7.2, R8.1
- net N$13: now also MDL1.RESET, R5.2; no longer JP4.1, MDL1.CH_PD
- net N$15: now also JP1.2; no longer JP2.1
- net N$17: now also MDL1.GPIO2, R6.1; no longer JP5.1, MDL1.RESET
- net N$9: now also MDL1.GPIO16; no longer MDL1.GPIO15
Routing:
- net VCC: track 0.00 -> 94.6 mm
- net VCC+3.3V: track 84.7 -> 0.00 mm
- net N$12: track 270.0 -> 191.0 mm
- net N$53: track 0.00 -> 78.9 mm
- net N$9: track 17.1 -> 79.4 mm
- net N$16: track 0.00 -> 15.9 mm
- net GND: track 163.8 -> 152.2 mm
- net N$18: track 0.00 -> 4.77 mm
- net N$14: track 11.2 -> 8.15 mm
- net N$11: track 32.4 -> 29.4 mm
- net 230FUSED: track 64.3 -> 61.6 mm
- net CURRENT: track 45.2 -> 42.5 mm
- net N$10: track 27.8 -> 25.5 mm
- net N$13: track 5.93 -> 3.90 mm
- net N$17: track 5.52 -> 3.88 mm
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
Commit message: Correction pcb
Parts:
- moved R8 6.64 mm to (11.9, 59.3), turned to 0 degrees
- moved U$3 0.18 mm to (35.2, 59.4), flipped to the bottom
Connections:
- net N$9 renamed DS18B20
- net GND: no longer R8.1
- net VCC: now also R8.1, U$3.3
Routing:
- net GND: track 152.2 -> 148.5 mm
- net VCC: track 94.6 -> 96.4 mm
- net N$16: track 15.9 -> 16.5 mm
- net DS18B20: track 79.4 -> 78.9 mm

Commit message: PCB finale
Parts:
- moved X1 2.19 mm to (28.7, 7.20)
- moved D2 1.94 mm to (53.2, 11.7)
- moved D1 1.92 mm to (48.6, 11.7)
- moved JP1 1.26 mm to (32.5, 77.1), turned to 0 degrees
- moved JP3 0.99 mm to (33.7, 69.7)
Routing:
- net NEUTRAL: track 48.2 -> 37.4 mm
- net 230OUT: track 12.6 -> 21.5 mm
- net 230IN: track 23.1 -> 31.0 mm
- net N$15: track 7.88 -> 11.3 mm
- net N$4: track 17.3 -> 15.1 mm
- net N$1: track 15.8 -> 13.8 mm
- net N$11: track 29.4 -> 30.6 mm
- net N$19: track 7.63 -> 8.65 mm
- net GND: track 148.5 -> 149.5 mm
- net N$14: track 8.15 -> 7.23 mm
- net PILOTE: track 13.6 -> 14.4 mm

Commit message: ...
Parts:
- added S1: (no value), switch-omron:B3F-10XX
- moved R4 6.26 mm to (35.5, 43.0)
- moved U$4 4.00 mm to (16.0, 40.9)
- moved R5 3.99 mm to (7.31, 76.2), turned to 270 degrees
- moved D2 3.91 mm to (51.5, 15.2)
- moved JP1 3.89 mm to (32.2, 81.0)
- moved D1 3.54 mm to (48.1, 15.2)
- moved C1 3.23 mm to (36.3, 54.4), turned to 180 degrees
- moved X1 2.56 mm to (31.2, 6.70)
- moved U$1 2.00 mm to (43.3, 36.9)
- moved IC1 2.00 mm to (33.8, 15.2), flipped to the bottom
- moved U$2 2.00 mm to (48.8, 36.9)
- moved F1 1.72 mm to (14.8, 16.1), turned to 315 degrees
- moved SV1 1.58 mm to (2.71, 66.1)
- moved R3 0.35 mm to (6.45, 66.5)
Connections:
- net 230IN: now also IC1.IP-, IC1.IP-@10, IC1.IP-@11, IC1.IP-@12, IC1.IP-@13, IC1.IP-@14, IC1.IP-@15, IC1.IP-@16, IC1.IP-@17, IC1.IP-@2, IC1.IP-@3, IC1.IP-@4, IC1.IP-@5, IC1.IP-@6, IC1.IP-@7, IC1.IP-@8, IC1.IP-@9; no longer IC1.IP+, IC1.IP+@10, IC1.IP+@11, IC1.IP+@12, IC1.IP+@13, IC1.IP+@14, IC1.IP+@15, IC1.IP+@16, IC1.IP+@17, IC1.IP+@2, IC1.IP+@3, IC1.IP+@4, IC1.IP+@5, IC1.IP+@6, IC1.IP+@7, IC1.IP+@8, IC1.IP+@9
- net 230OUT: now also IC1.IP+, IC1.IP+@10, IC1.IP+@11, IC1.IP+@12, IC1.IP+@13, IC1.IP+@14, IC1.IP+@15, IC1.IP+@16, IC1.IP+@17, IC1.IP+@2, IC1.IP+@3, IC1.IP+@4, IC1.IP+@5, IC1.IP+@6, IC1.IP+@7, IC1.IP+@8, IC1.IP+@9; no longer IC1.IP-, IC1.IP-@10, IC1.IP-@11, IC1.IP-@12, IC1.IP-@13, IC1.IP-@14, IC1.IP-@15, IC1.IP-@16, IC1.IP-@17, IC1.IP-@2, IC1.IP-@3, IC1.IP-@4, IC1.IP-@5, IC1.IP-@6, IC1.IP-@7, IC1.IP-@8, IC1.IP-@9
- net GND: now also S1.3, S1.4
- net N$13: now also S1.2
Routing:
- net GND: track 149.5 -> 102.1 mm, vias 0 -> 5
- net 230FUSED: track 61.6 -> 45.6 mm
- net DS18B20: track 78.5 -> 64.0 mm
- net 230OUT: track 21.5 -> 11.0 mm
- net NEUTRAL: track 37.4 -> 47.4 mm
- net N$13: track 3.90 -> 11.9 mm
- net 230IN: track 31.0 -> 24.1 mm
- net CURRENT: track 42.5 -> 47.5 mm
- net N$53: track 78.9 -> 83.1 mm
- net N$14: track 7.23 -> 11.1 mm
- net N$1: track 13.8 -> 10.3 mm
- net N$15: track 11.3 -> 14.5 mm
- net N$4: track 15.1 -> 12.3 mm
- net PILOTE: track 14.4 -> 11.8 mm
- net N$12: track 191.0 -> 193.3 mm
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Other:
- board size 56 x 79 mm -> 16 x 2 mm
